Commit message: tweeked xacro

File: description/lidar.xacro (robot description, xacro)
@@ -4,5 +4,5 @@
         <parent link="chassis"/>
         <child link="laser_frame"/>
-        <origin xyz="0.122 0 0.212" rpy="0 0 0"/>
+        <origin xyz="0.72 0 0.32" rpy="0 0 0"/>
     </joint>
     <link name="laser_frame">

File: description/robot_core.xacro (robot description, xacro)
@@ -67,5 +67,5 @@
     </link>
     <gazebo reference="chassis">
-        <material>Gazebo/Orange</material>
+        <material>Gazebo/Red</material>
     </gazebo>
     <!-- LEFT WHEEL LINK -->

Commit message: rplidar mesh test

File: description/lidar.xacro (robot description, xacro)
@@ -9,12 +9,6 @@
         <visual>
             <geometry>
-                <cylinder radius="0.05" length="0.04"/>
-            </geometry>
-            <material name="black"/>
-        </visual>
-        <visual>
-            <origin xyz="0 0 -0.05"/>
-            <geometry>
-                <cylinder radius="0.01" length="0.1"/>
+                <box size="0.1 0.1 0.1"/>
+				<meshfile name="rplidar.dae" scale="0.001 0.001 0.001" />
             </geometry>
             <material name="black"/>

File: description/rplidar.urdf.xacro (robot description, xacro)
@@ -8,11 +8,11 @@
 			</geometry>
 		</collision>
-		<vision>
-			<origin xyz="0 0 -0.03125" rpy="1.5707 0 0"/>
+		<visual>
+			<origin xyz="0 0 -0.03125" rpy="0 0 0"/>
 			<geometry>
 				<box size="0.1 0.1 0.1"/>
-				<meshfile name="package://BLAHPACKAGENAME/meshes/rplidar.dae" scale="0.001 0.001 0.001" />
+				<meshfile name="rplidar.dae" scale="0.001 0.001 0.001" />
 			</geometry>
-		</vision>
+		</visual>
 		<inertial>
 			<mass value="1e-5"/>
@@ -24,5 +24,5 @@
 		<axis xyz="0 1 0"/>
 		<origin xyz="0 0 0.035" rpy="0 0 0 "/>
-		<parent link="plate_top_link"/>
+		<parent link="chassis_link"/>
 		<child link="rplidar_link"/>
 	</joint>

Commit message: rplidar urdf edit

File: description/lidar.xacro (robot description, xacro)
@@ -4,10 +4,10 @@
         <parent link="chassis"/>
         <child link="laser_frame"/>
-        <origin xyz="0.72 0 0.32" rpy="0 0 0"/>
+        <origin xyz="0.72 0 0.22" rpy="0 0 0"/>
     </joint>
     <link name="laser_frame">
         <visual>
             <geometry>
-                <box size="0.1 0.1 0.1"/>
+                <!-- <box size="0.1 0.1 0.1"/> -->
 				<meshfile name="rplidar.dae" scale="0.001 0.001 0.001" />
             </geometry>

Commit message: ros2 update from old data line

File: description/lidar.xacro (robot description, xacro)
@@ -10,5 +10,5 @@
             <geometry>
                 <!-- <box size="0.1 0.1 0.1"/> -->
-				<meshfile name="rplidar.dae" scale="0.001 0.001 0.001" />
+				<mesh filename="rplidar.dae" scale="0.001 0.001 0.001" />
             </geometry>
             <material name="black"/>

Commit message: fixed what I broke

File: description/lidar.xacro (robot description, xacro)
@@ -4,11 +4,11 @@
         <parent link="chassis"/>
         <child link="laser_frame"/>
-        <origin xyz="0.72 0 0.22" rpy="0 0 0"/>
+        <origin xyz="0.72 0 0.28" rpy="0 0 0"/>
     </joint>
     <link name="laser_frame">
         <visual>
             <geometry>
-                <!-- <box size="0.1 0.1 0.1"/> -->
-				<mesh filename="rplidar.dae" scale="0.001 0.001 0.001" />
+                <box size="0.1 0.1 0.1"/>
+				<!-- <mesh filename="rplidar.dae" scale="0.001 0.001 0.001" /> -->
             </geometry>
             <material name="black"/>

Commit message: Update lidar.xacro
back to cylinder

File: description/lidar.xacro (robot description, xacro)
@@ -4,11 +4,11 @@
         <parent link="chassis"/>
         <child link="laser_frame"/>
-        <origin xyz="0.72 0 0.28" rpy="0 0 0"/>
+        <origin xyz="0.72 0 0.22" rpy="0 0 0"/>
     </joint>
     <link name="laser_frame">
         <visual>
             <geometry>
-                <box size="0.1 0.1 0.1"/>
-				<!-- <mesh filename="rplidar.dae" scale="0.001 0.001 0.001" /> -->
+                <cylinder radius="0.05" length="0.04"/>
+				<!-- <mesh filename="rplidar_a1.dae" scale="0.001 0.001 0.001" /> -->
             </geometry>
             <material name="black"/>
