Commit message: cleaned  up description to be  more like  the real dimentions  and  colors

File: description/face.xacro (robot description, xacro)
@@ -26,5 +26,5 @@
                 <cylinder radius="0.05" length="0.02"/>
             </geometry>
-            <material name="red"/>
+            <material name="black"/>
         </visual>
     </link>

File: description/lidar.xacro (robot description, xacro)
@@ -4,10 +4,10 @@
         <parent link="chassis"/>
         <child link="laser_frame"/>
-        <origin xyz="0.72 0 0.22" rpy="0 0 0"/>
+        <origin xyz="0.65 0 0.18" rpy="0 0 0"/>
     </joint>
     <link name="laser_frame">
         <visual>
             <geometry>
-                <cylinder radius="0.05" length="0.04"/>
+                <cylinder radius="0.035" length="0.02"/>
 				<!-- <mesh filename="rplidar_a1.dae" scale="0.001 0.001 0.001" /> -->
             </geometry>
@@ -16,8 +16,8 @@
         <collision>
             <geometry>
-                <cylinder radius="0.05" length="0.04"/>
+                <cylinder radius="0.035" length="0.02"/>
             </geometry>
         </collision>
-        <xacro:inertial_cylinder mass="0.1" length="0.04" radius="0.05">
+        <xacro:inertial_cylinder mass="0.1" length="0.02" radius="0.035">
             <origin xyz="0 0 0" rpy="0 0 0"/>
         </xacro:inertial_cylinder>

File: description/robot_core.xacro (robot description, xacro)
@@ -2,17 +2,17 @@
 <robot xmlns:xacro="http://www.ros.org/wiki/xacro" >
     <xacro:include filename="inertial_macros.xacro"/>
-    <xacro:property name="chassis_length" value="0.88"/>
-    <xacro:property name="chassis_width" value="0.40"/>
-    <xacro:property name="chassis_height" value="0.15"/>
+    <xacro:property name="chassis_length" value="0.65"/>
+    <xacro:property name="chassis_width" value="0.44"/>
+    <xacro:property name="chassis_height" value="0.165"/>
     <xacro:property name="chassis_mass" value="1.0"/>
-    <xacro:property name="wheel_radius" value="0.10"/>
-    <xacro:property name="wheel_thickness" value="0.05"/>
+    <xacro:property name="wheel_radius" value="0.13"/>
+    <xacro:property name="wheel_thickness" value="0.07"/>
     <xacro:property name="wheel_mass" value="0.05"/>
-    <xacro:property name="wheel_offset_x" value="0.5"/>
+    <xacro:property name="wheel_offset_x" value="0.48"/>
     <xacro:property name="wheel_offset_y" value="0.255"/>
     <xacro:property name="wheel_offset_z" value="0.01"/>
-    <xacro:property name="caster_wheel_radius" value="0.10"/>
+    <xacro:property name="caster_wheel_radius" value="0.13"/>
     <xacro:property name="caster_wheel_mass" value="0.01"/>
-    <xacro:property name="caster_wheel_offset_x" value="0.075"/>
+    <xacro:property name="caster_wheel_offset_x" value="0.01"/>
     <xacro:property name="caster_wheel_offset_z" value="${wheel_offset_z - wheel_radius + caster_wheel_radius}"/>
     <material name="white">
@@ -27,4 +27,7 @@
     <material name="black">
         <color rgba="0 0 0 1"/>
+    </material>
+    <material name="grey">
+        <color rgba="0.5 0.5 0.5 1"/>
     </material>
     <material name="red">
@@ -54,5 +57,5 @@
                 <box size="${chassis_length} ${chassis_width} ${chassis_height}"/>
             </geometry>
-            <material name="orange"/>
+            <material name="red"/>
         </visual>
         <collision>
@@ -81,5 +84,5 @@
                 <cylinder radius="${wheel_radius}" length="${wheel_thickness}"/>
             </geometry>
-            <material name="blue"/>
+            <material name="grey"/>
         </visual>
         <collision>
@@ -93,5 +96,5 @@
     </link>
     <gazebo reference="left_wheel">
-        <material>Gazebo/Blue</material>
+        <material>Gazebo/Grey</material>
     </gazebo>
     <!-- RIGHT WHEEL LINK -->
@@ -107,5 +110,5 @@
                 <cylinder radius="${wheel_radius}" length="${wheel_thickness}"/>
             </geometry>
-            <material name="blue"/>
+            <material name="grey"/>
         </visual>
         <collision>
@@ -119,5 +122,5 @@
     </link>
     <gazebo reference="right_wheel">
-        <material>Gazebo/Blue</material>
+        <material>Gazebo/Grey</material>
     </gazebo>
     <!-- CASTER WHEEL LINK -->
@@ -132,5 +135,5 @@
                 <sphere radius="${caster_wheel_radius}"/>
             </geometry>
-            <material name="white"/>
+            <material name="grey"/>
         </visual>
         <collision>
@@ -144,5 +147,5 @@
     </link>
     <gazebo reference="caster_wheel">
-        <material>Gazebo/White</material>
+        <material>Gazebo/Grey</material>
         <mu1 value="0.001"/>
         <mu2 value="0.001"/>
