Commit message: fixed typo

File: description/robot_core.xacro (robot description, xacro)
@@ -10,5 +10,5 @@
     <xacro:property name="wheel_mass" value="0.05"/>
     <xacro:property name="wheel_offset_x" value="0.5"/>
-    <xacro:property name="wheel_offset_y" value="0.25.5"/>
+    <xacro:property name="wheel_offset_y" value="0.255"/>
     <xacro:property name="wheel_offset_z" value="0.01"/>
     <xacro:property name="caster_wheel_radius" value="0.10"/>

Commit message: Update robot_core.xacro
edit to niagra dimentions

File: description/robot_core.xacro (robot description, xacro)
@@ -2,17 +2,17 @@
 <robot xmlns:xacro="http://www.ros.org/wiki/xacro" >
     <xacro:include filename="inertial_macros.xacro"/>
-    <xacro:property name="chassis_length" value="0.65"/>
-    <xacro:property name="chassis_width" value="0.44"/>
-    <xacro:property name="chassis_height" value="0.165"/>
+    <xacro:property name="chassis_length" value="0.95"/>
+    <xacro:property name="chassis_width" value="0.55"/>
+    <xacro:property name="chassis_height" value="0.18"/>
     <xacro:property name="chassis_mass" value="1.0"/>
-    <xacro:property name="wheel_radius" value="0.13"/>
-    <xacro:property name="wheel_thickness" value="0.07"/>
+    <xacro:property name="wheel_radius" value="0.12"/>
+    <xacro:property name="wheel_thickness" value="0.08"/>
     <xacro:property name="wheel_mass" value="0.05"/>
-    <xacro:property name="wheel_offset_x" value="0.48"/>
-    <xacro:property name="wheel_offset_y" value="0.255"/>
+    <xacro:property name="wheel_offset_x" value="0.25"/>
+    <xacro:property name="wheel_offset_y" value="0.18"/>
     <xacro:property name="wheel_offset_z" value="0.01"/>
     <xacro:property name="caster_wheel_radius" value="0.13"/>
     <xacro:property name="caster_wheel_mass" value="0.01"/>
-    <xacro:property name="caster_wheel_offset_x" value="0.01"/>
+    <xacro:property name="caster_wheel_offset_x" value="0.90"/>
     <xacro:property name="caster_wheel_offset_z" value="${wheel_offset_z - wheel_radius + caster_wheel_radius}"/>
     <material name="white">
